File: hardware/RevA/RevA.kicad_pcb (KiCad board)
At the start: 4 copper layers, 85 x 54 mm, 143 parts, among them J1 USB_C_Receptacle_USB2.0, J2 DNP Conn_02x02_Odd_Even, J3 DNP Conn_01x02, J4 DNP Conn_02x03_Odd_Even, J5 DNP Conn_01x02, SW1 SW_Push, SW2 SW_Push, U1 SY8120B1ABC, U10 SPI RAM LY68L6400SLIT, U2 XC6206P25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

Commit message: RevA 0.2 updates
Parts:
- added R36: 1K, Resistor_SMD:R_0402_1005Metric, F.Cu at (131.2, 63.6)
- added R37: 1K, Resistor_SMD:R_0402_1005Metric, F.Cu at (131.2, 65.6)
- C11, C14: value 4p7 -> 20p
- moved TP1 2.86 mm to (129.2, 63.6)
- moved TP2 0.07 mm to (129.2, 65.6)
Routing:
- net +3V3: track 129.5 -> 112.4 mm, vias 41 -> 43
- net GND: track 158.2 -> 151.4 mm
- net /ALT0_FLEXSPI_B_DQS: track 26.4 -> 22.9 mm, vias 0 -> 2
- net /ALT0_LPUART1_TXD: track 17.8 -> 18.9 mm
- net /ALT0_LPUART1_RXD: track 21.0 -> 21.9 mm
