File: hardware/RevB/RevB.kicad_pcb (KiCad board)
At the start: 4 copper layers, 93.7 x 54 mm, 100 parts, among them J1 USB_C_Receptacle_USB2.0, J2 DNP Conn_02x02_Odd_Even, J3 DNP Conn_01x02, J4 DNP Conn_02x03_Odd_Even, J5 DNP Conn_01x02, J6 Conn_ULX3S, SW1 SW_Push, SW2 SW_Push, U1 SY8120B1ABC, U10 SPI RAM LY68L6400SLIT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

Commit message: Fix weird via
Routing:
- net VBUS: vias 22 -> 23
- net (no net): vias 4 -> 3

Commit message: progress
Parts:
- removed LOGO2: Logo_Open_Hardware_Small, ecp5board:logo
- moved C10 50.4 mm to (120.6, 68.8)
- moved C5 50.4 mm to (120.6, 64.8)
- moved C9 50.4 mm to (123.5, 64.8)
- moved C8 50.4 mm to (120.6, 66.8)
- moved C11 50.4 mm to (123.5, 66.8)
- moved LOGO3 1.70 mm to (176.0, 62.2)

Commit message: Update BOM
Other:
- board text added: "PERGOLA RevB 0.1-WIP"

Commit message: Routing WIP experiment
Parts:
- added LOGO2: Logo_Open_Hardware_Small, ecp5board:logo, F.Cu at (169.0, 74.0)
- R10: value 18k -> 18k 1%
- R11, R9: value 15k -> 15k 1%
- R12: value 3k3 -> 3k3 1%
- moved C41 43.1 mm to (209.0, 82.0)
- moved C44 42.6 mm to (208.0, 72.5), turned to 270 degrees
- moved U7 41.5 mm to (203.0, 81.0)
- moved U10 40.5 mm to (202.0, 72.0)
Connections:
- J6 pad 10: (no net) -> /G2+
- J6 pad 11: (no net) -> /G3-
- J6 pad 12: (no net) -> /G3+
- J6 pad 13: (no net) -> /G4-
- J6 pad 14: (no net) -> /G4+
- J6 pad 15: (no net) -> /G5-
- J6 pad 16: (no net) -> /G5+
- J6 pad 17: (no net) -> /G6-
- J6 pad 18: (no net) -> /G6+
- J6 pad 23: (no net) -> /G7-
- J6 pad 24: (no net) -> /G7+
- J6 pad 25: (no net) -> /G8-
- J6 pad 26: (no net) -> /G8+
- J6 pad 27: (no net) -> /G9-
- J6 pad 28: (no net) -> /G9+
- J6 pad 29: (no net) -> /G10-
- J6 pad 30: (no net) -> /G10+
- J6 pad 31: (no net) -> /G11-
- J6 pad 32: (no net) -> /G11+
- J6 pad 33: (no net) -> /G12-
- J6 pad 34: (no net) -> /G12+
- J6 pad 35: (no net) -> /G13-
- J6 pad 36: (no net) -> /G13+
- J6 pad 5: (no net) -> /G0-
- J6 pad 6: (no net) -> /G0+
- J6 pad 7: (no net) -> /G1-
- J6 pad 8: (no net) -> /G1+
- J6 pad 9: (no net) -> /G2-
- RN7 pad 1: /PMOD4_1x -> (no net)
- RN7 pad 2: /PMOD4_5x -> (no net)
- RN7 pad 3: /PMOD4_2x -> (no net)
- RN7 pad 4: /PMOD4_6x -> (no net)
- RN8 pad 1: /PMOD4_3x -> (no net)
- RN8 pad 2: /PMOD4_7x -> (no net)
- RN8 pad 3: /PMOD4_4x -> (no net)
- RN8 pad 4: /PMOD4_8x -> (no net)
- U10 pad 1: /RAM2_~CS~ -> (no net)
- U10 pad 2: /RAM2_D1 -> (no net)
- U10 pad 3: /RAM2_D2 -> (no net)
- U10 pad 5: /RAM2_D0 -> (no net)
- U10 pad 6: /RAM2_CLK -> (no net)
- U10 pad 7: /RAM2_D3 -> (no net)
- U7 pad 1: /RAM1_~CS~ -> (no net)
- U7 pad 2: /RAM1_D1 -> (no net)
- U7 pad 3: /RAM1_D2 -> (no net)
- U7 pad 5: /RAM1_D0 -> (no net)
- U7 pad 6: /RAM1_CLK -> (no net)
- U7 pad 7: /RAM1_D3 -> (no net)
- U8 pad A10: /RAM1_D1 -> /G7-
- U8 pad A11: /RAM1_D2 -> /G4+
- U8 pad A12: /PMOD4_5x -> /G4-
- U8 pad A13: /PMOD4_6x -> /G1+
- U8 pad A14: /PMOD4_7x -> /G1-
- U8 pad A15: /PMOD4_8x -> /G0-
- U8 pad A2: /RAM2_~CS~ -> /G13+
- U8 pad A3: /RAM2_D3 -> /G12+
- U8 pad A4: /RAM2_CLK -> /G12-
- U8 pad A5: /RAM2_D0 -> /G10+
- U8 pad A6: (no net) -> /G10-
- U8 pad A9: /RAM1_~CS~ -> /G7+
- U8 pad B10: /RAM1_D0 -> /G6+
- U8 pad B11: /PMOD4_1x -> /G5+
- U8 pad B12: /PMOD4_2x -> /G3+
- U8 pad B13: /PMOD4_3x -> /G2+
- U8 pad B14: /PMOD4_4x -> /G0+
- U8 pad B3: /RAM2_D1 -> /G13-
- U8 pad B4: /RAM2_D2 -> /G11-
- U8 pad B8: /RAM1_D3 -> /G9-
- U8 pad B9: /RAM1_CLK -> /G8+
- U8 pad C10: (no net) -> /G6-
- U8 pad C11: (no net) -> /G5-
- U8 pad C12: (no net) -> /G3-
- U8 pad C13: (no net) -> /G2-
- U8 pad C4: (no net) -> /G11+
- U8 pad C8: (no net) -> /G9+
- U8 pad C9: (no net) -> /G8-
Routing:
- net /G11+: track 0.00 -> 38.2 mm, vias 0 -> 2
- net /G0+: track 0.00 -> 38.1 mm
- net /G9+: track 0.00 -> 37.6 mm
- net /G13+: track 0.00 -> 37.5 mm
- net /G2-: track 0.00 -> 37.1 mm, vias 0 -> 2
- net /G12+: track 0.00 -> 36.9 mm
- net /G1+: track 0.00 -> 36.8 mm
- net /G0-: track 0.00 -> 36.7 mm
- net /G2+: track 0.00 -> 36.4 mm, vias 0 -> 2
- net /G1-: track 0.00 -> 36.3 mm
- net /G3-: track 0.00 -> 35.9 mm, vias 0 -> 2
- net /G9-: track 0.00 -> 35.9 mm
- net /G8+: track 0.00 -> 35.8 mm, vias 0 -> 1
- net /G10+: track 0.00 -> 35.4 mm
- net /G3+: track 0.00 -> 35.4 mm
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