File: hardware/RevB/RevB.sch (KiCad schematic (older format))
At the start: 100 parts, among them J1 USB_C_Receptacle_USB2.0, J2 DNP Conn_02x02_Odd_Even, J3 DNP Conn_01x02, J4 DNP Conn_02x03_Odd_Even, J5 DNP Conn_01x02, J6 Conn_ULX3S, SW1 SW_Push, SW2 SW_Push, U1 SY8120B1ABC, U10 SPI RAM LY68L6400SLIT, U2 XC6206P25, U3 SY8120B1ABC, U4 SPI Flash W25Q128JVSIQ, U5 USBLC6-2P6, U6 ATSAMD21G18A-AUT, U7 SPI RAM LY68L6400SLIT, U8 LFE5U-12F-6BG256C, U9 16MHz 20ppm

Commit message: Update BOM
Parts:
- C10, C11, C2, C30, C31, C32, C33, C34, C35, C36, C37, C38, C39, C41, C42, C44, C5, C8, C9: LCSC https://lcsc.com/product-detail/Multilayer-Ceramic-Capacito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 -> (none)
- R10: value 18k -> 18k 1%
- R11, R9: value 15k -> 15k 1%
- R12: value 3k3 -> 3k3 1%
Changed lines of the file:
@@
 P 3600 1800
 F 0 "R9" H 3550 1950 50  0000 C CNN
-F 1 "15k" V 3600 1800 39  0000 C CNN
+F 1 "15k 1%" V 3700 1800 39  0000 C CNN
 F 2 "Resistor_SMD:R_0402_1005Metric" V 3530 1800 50  0001 C CNN
 F 3 " " H 3600 1800 50  0001 C CNN
@@
 P 3600 2300
 F 0 "R10" H 3500 2450 50  0000 C CNN
-F 1 "18k" V 3600 2300 39  0000 C CNN
+F 1 "18k 1%" V 3700 2300 39  0000 C CNN
 F 2 "Resistor_SMD:R_0402_1005Metric" V 3530 2300 50  0001 C CNN
 F 3 " " H 3600 2300 50  0001 C CNN
@@
 P 3600 6200
 F 0 "R12" H 3500 6350 50  0000 C CNN
-F 1 "3k3" V 3600 6200 39  0000 C CNN
+F 1 "3k3 1%" V 3700 6200 39  0000 C CNN
 F 2 "Resistor_SMD:R_0402_1005Metric" V 3530 6200 50  0001 C CNN
 F 3 " " H 3600 6200 50  0001 C CNN
@@
 P 3600 5700
 F 0 "R11" H 3500 5850 50  0000 C CNN
-F 1 "15k" V 3600 5700 39  0000 C CNN
+F 1 "15k 1%" V 3700 5700 39  0000 C CNN
 F 2 "Resistor_SMD:R_0402_1005Metric" V 3530 5700 50  0001 C CNN
 F 3 " " H 3600 5700 50  0001 C CNN
@@
 F 2 "Capacitor_SMD:C_0402_1005Metric" H 19750 12200 50  0001 C CNN
 F 3 " " H 19750 12200 50  0001 C CNN
-F 4 "https://lcsc.com/product-detail/Multilayer-Ceramic-Capacitors-MLCC-SMD-SMT_SAMSUNG_CL21A226MOQNNNE_22uF-226-20-16V_C98190.html" H 19750 12200 50  0001 C CNN "LCSC"
+F 4 "" H 19750 12200 50  0001 C CNN "LCSC"
 	1    19750 12200
 	-1   0    0    1
@@
 F 2 "Capacitor_SMD:C_0402_1005Metric" H 20100 12200 50  0001 C CNN
 F 3 " " H 20100 12200 50  0001 C CNN
-F 4 "https://lcsc.com/product-detail/Multilayer-Ceramic-Capacitors-MLCC-SMD-SMT_SAMSUNG_CL21A226MOQNNNE_22uF-226-20-16V_C98190.html" H 20100 12200 50  0001 C CNN "LCSC"
+F 4 "" H 20100 12200 50  0001 C CNN "LCSC"
 	1    20100 12200
 	-1   0    0    1
@@
 F 2 "Capacitor_SMD:C_0402_1005Metric" H 20450 12200 50  0001 C CNN
 F 3 " " H 20450 12200 50  0001 C CNN
-F 4 "https://lcsc.com/product-detail/Multilayer-Ceramic-Capacitors-MLCC-SMD-SMT_SAMSUNG_CL21A226MOQNNNE_22uF-226-20-16V_C98190.html" H 20450 12200 50  0001 C CNN "LCSC"
+F 4 "" H 20450 12200 50  0001 C CNN "LCSC"
 	1    20450 12200
 	-1   0    0    1
@@
 F 2 "Capacitor_SMD:C_0402_1005Metric" H 20800 12200 50  0001 C CNN
 F 3 " " H 20800 12200 50  0001 C CNN
-F 4 "https://lcsc.com/product-detail/Multilayer-Ceramic-Capacitors-MLCC-SMD-SMT_SAMSUNG_CL21A226MOQNNNE_22uF-226-20-16V_C98190.html" H 20800 12200 50  0001 C CNN "LCSC"
+F 4 "" H 20800 12200 50  0001 C CNN "LCSC"
 	1    20800 12200
 	-1   0    0    1
@@
 F 2 "Capacitor_SMD:C_0402_1005Metric" H 21150 12200 50  0001 C CNN
 F 3 " " H 21150 12200 50  0001 C CNN
-F 4 "https://lcsc.com/product-detail/Multilayer-Ceramic-Capacitors-MLCC-SMD-SMT_SAMSUNG_CL21A226MOQNNNE_22uF-226-20-16V_C98190.html" H 21150 12200 50  0001 C CNN "LCSC"
+F 4 "" H 21150 12200 50  0001 C CNN "LCSC"
 	1    21150 12200
 	-1   0    0    1
@@
 F 2 "Capacitor_SMD:C_0402_1005Metric" H 19750 13050 50  0001 C CNN
 F 3 " " H 19750 13050 50  0001 C CNN
-F 4 "https://lcsc.com/product-detail/Multilayer-Ceramic-Capacitors-MLCC-SMD-SMT_SAMSUNG_CL21A226MOQNNNE_22uF-226-20-16V_C98190.html" H 19750 13050 50  0001 C CNN "LCSC"
+F 4 "" H 19750 13050 50  0001 C CNN "LCSC"
 	1    19750 13050
 	-1   0    0    1
@@
 F 2 "Capacitor_SMD:C_0402_1005Metric" H 20100 13050 50  0001 C CNN
 F 3 " " H 20100 13050 50  0001 C CNN
-F 4 "https://lcsc.com/product-detail/Multilayer-Ceramic-Capacitors-MLCC-SMD-SMT_SAMSUNG_CL21A226MOQNNNE_22uF-226-20-16V_C98190.html" H 20100 13050 50  0001 C CNN "LCSC"
+F 4 "" H 20100 13050 50  0001 C CNN "LCSC"
 	1    20100 13050
 	-1   0    0    1
@@
 F 2 "Capacitor_SMD:C_0402_1005Metric" H 19750 13850 50  0001 C CNN
 F 3 " " H 19750 13850 50  0001 C CNN
-F 4 "https://lcsc.com/product-detail/Multilayer-Ceramic-Capacitors-MLCC-SMD-SMT_SAMSUNG_CL21A226MOQNNNE_22uF-226-20-16V_C98190.html" H 19750 13850 50  0001 C CNN "LCSC"
+F 4 "" H 19750 13850 50  0001 C CNN "LCSC"
 	1    19750 13850
 	-1   0    0    1
@@
 F 2 "Capacitor_SMD:C_0402_1005Metric" H 20100 13850 50  0001 C CNN
 F 3 " " H 20100 13850 50  0001 C CNN
-F 4 "https://lcsc.com/product-detail/Multilayer-Ceramic-Capacitors-MLCC-SMD-SMT_SAMSUNG_CL21A226MOQNNNE_22uF-226-20-16V_C98190.html" H 20100 13850 50  0001 C CNN "LCSC"
+F 4 "" H 20100 13850 50  0001 C CNN "LCSC"
 	1    20100 13850
 	-1   0    0    1
@@
 F 2 "Capacitor_SMD:C_0402_1005Metric" H 20450 13850 50  0001 C CNN
 F 3 " " H 20450 13850 50  0001 C CNN
-F 4 "https://lcsc.com/product-detail/Multilayer-Ceramic-Capacitors-MLCC-SMD-SMT_SAMSUNG_CL21A226MOQNNNE_22uF-226-20-16V_C98190.html" H 20450 13850 50  0001 C CNN "LCSC"
+F 4 "" H 20450 13850 50  0001 C CNN "LCSC"
 	1    20450 13850
 	-1   0    0    1
@@
 F 2 "Capacitor_SMD:C_0402_1005Metric" H 14900 8650 50  0001 C CNN
 F 3 " " H 14900 8650 50  0001 C CNN
-F 4 "https://lcsc.com/product-detail/Multilayer-Ceramic-Capacitors-MLCC-SMD-SMT_SAMSUNG_CL21A226MOQNNNE_22uF-226-20-16V_C98190.html" H 14900 8650 50  0001 C CNN "LCSC"
+F 4 "" H 14900 8650 50  0001 C CNN "LCSC"
 	1    14900 8650
 	-1   0    0    1
@@
 F 2 "Capacitor_SMD:C_0402_1005Metric" H 15000 4800 50  0001 C CNN
 F 3 " " H 15000 4800 50  0001 C CNN
-F 4 "https://lcsc.com/product-detail/Multilayer-Ceramic-Capacitors-MLCC-SMD-SMT_SAMSUNG_CL21A226MOQNNNE_22uF-226-20-16V_C98190.html" H 15000 4800 50  0001 C CNN "LCSC"
+F 4 "" H 15000 4800 50  0001 C CNN "LCSC"
 	1    15000 4800
 	-1   0    0    1
@@
 F 2 "Capacitor_SMD:C_0402_1005Metric" H 14900 10150 50  0001 C CNN
 F 3 " " H 14900 10150 50  0001 C CNN
-F 4 "https://lcsc.com/product-detail/Multilayer-Ceramic-Capacitors-MLCC-SMD-SMT_SAMSUNG_CL21A226MOQNNNE_22uF-226-20-16V_C98190.html" H 14900 10150 50  0001 C CNN "LCSC"
+F 4 "" H 14900 10150 50  0001 C CNN "LCSC"
 	1    14900 10150
 	-1   0    0    1
@@
 F 2 "Capacitor_SMD:C_0402_1005Metric" H 15050 7100 50  0001 C CNN
 F 3 " " H 15050 7100 50  0001 C CNN
-F 4 "https://lcsc.com/product-detail/Multilayer-Ceramic-Capacitors-MLCC-SMD-SMT_SAMSUNG_CL21A226MOQNNNE_22uF-226-20-16V_C98190.html" H 15050 7100 50  0001 C CNN "LCSC"
+F 4 "" H 15050 7100 50  0001 C CNN "LCSC"
 	1    15050 7100
 	-1   0    0    1
@@
 F 2 "Capacitor_SMD:C_0402_1005Metric" H 6100 11050 50  0001 C CNN
 F 3 " " H 6100 11050 50  0001 C CNN
-F 4 "https://lcsc.com/product-detail/Multilayer-Ceramic-Capacitors-MLCC-SMD-SMT_SAMSUNG_CL21A226MOQNNNE_22uF-226-20-16V_C98190.html" H 6100 11050 50  0001 C CNN "LCSC"
+F 4 "" H 6100 11050 50  0001 C CNN "LCSC"
 	1    6100 11050
 	-1   0    0    1
@@
 F 2 "Capacitor_SMD:C_0402_1005Metric" H 7450 10950 50  0001 C CNN
 F 3 " " H 7450 10950 50  0001 C CNN
-F 4 "https://lcsc.com/product-detail/Multilayer-Ceramic-Capacitors-MLCC-SMD-SMT_SAMSUNG_CL21A226MOQNNNE_22uF-226-20-16V_C98190.html" H 7450 10950 50  0001 C CNN "LCSC"
+F 4 "" H 7450 10950 50  0001 C CNN "LCSC"
 	1    7450 10950
 	-1   0    0    1
@@
 F 2 "Capacitor_SMD:C_0402_1005Metric" H 7800 10950 50  0001 C CNN
 F 3 " " H 7800 10950 50  0001 C CNN
-F 4 "https://lcsc.com/product-detail/Multilayer-Ceramic-Capacitors-MLCC-SMD-SMT_SAMSUNG_CL21A226MOQNNNE_22uF-226-20-16V_C98190.html" H 7800 10950 50  0001 C CNN "LCSC"
+F 4 "" H 7800 10950 50  0001 C CNN "LCSC"
 	1    7800 10950
 	-1   0    0    1
@@
 F 2 "Capacitor_SMD:C_0402_1005Metric" H 8150 10950 50  0001 C CNN
 F 3 " " H 8150 10950 50  0001 C CNN
-F 4 "https://lcsc.com/product-detail/Multilayer-Ceramic-Capacitors-MLCC-SMD-SMT_SAMSUNG_CL21A226MOQNNNE_22uF-226-20-16V_C98190.html" H 8150 10950 50  0001 C CNN "LCSC"
+F 4 "" H 8150 10950 50  0001 C CNN "LCSC"
 	1    8150 10950
 	-1   0    0    1
@@
 F 2 "Capacitor_SMD:C_0402_1005Metric" H 8500 10950 50  0001 C CNN
 F 3 " " H 8500 10950 50  0001 C CNN
-F 4 "https://lcsc.com/product-detail/Multilayer-Ceramic-Capacitors-MLCC-SMD-SMT_SAMSUNG_CL21A226MOQNNNE_22uF-226-20-16V_C98190.html" H 8500 10950 50  0001 C CNN "LCSC"
+F 4 "" H 8500 10950 50  0001 C CNN "LCSC"
 	1    8500 10950
 	-1   0    0    1

Commit message: Routing WIP experiment
Connections:
- net labels added: G0+, G0-, G1+, G1-, G10+, G10-, G11+, G11-, G12+, G12-, G13+, G13-, G2+, G2-, G3+, G3-, G4+, G4-, G5+, G5-, G6+, G6-, G7+, G7-, G8+, G8-, G9+, G9-
- wire segments 658 -> 722
- no-connect marks 154 -> 120
Other:
- moved on the sheet: C5
